File: eagle_files/SKL5/mainbrd.brd (EAGLE design)
At the start: 54 x 42.2 mm, 20 parts

Commit message: more thin on the left
Parts:
- moved JP2 9.25 mm to (5.08, 25.4)
- moved R7 8.25 mm to (6.99, 31.8)
- moved R5 5.08 mm to (9.53, 36.8)
- moved R6 5.08 mm to (5.71, 36.8)
- moved JP3 1.27 mm to (5.08, 17.8)
Routing:
- net VIN: track 52.0 -> 60.8 mm
- net 5V: track 139.3 -> 145.2 mm
- net SDA: track 67.6 -> 70.8 mm
- net SCL: track 62.7 -> 65.0 mm
- net GND: track 154.9 -> 156.6 mm
Other:
- board size 54 x 42.2 mm -> 51.4 x 41.6 mm

Commit message: thicker bois
Routing:
- net SDA: track 70.8 -> 71.6 mm
- net VIN: track 60.8 -> 60.0 mm

Commit message: fixes
Connections:
- net 5V: now also U$1.1; no longer U$1.4
- net GND: now also U$1.2; no longer U$1.1
- net SCL: now also U$1.3; no longer U$1.2
- net SDA: now also U$1.4; no longer U$1.3
Routing:
- net 5V: track 145.2 -> 151.5 mm, vias 1 -> 3
- net GND: track 156.6 -> 158.7 mm
- net VIN: track 60.0 -> 58.1 mm
- net SCL: track 65.4 -> 67.0 mm
- net SDA: track 71.6 -> 72.4 mm
Other:
- board text added: "J PODOLAK SKL5 2020"
